File: hardware/diy_atx_psu.kicad_sch (KiCad schematic)
At the start: 21 parts, among them J1 ATX SIGNAL MAP ONLY, J2 RED +12V, J3 YELLOW +5V, J4 GREEN +3.3V, J5 BLACK COM, J6 ADJ +, J7 ADJ - / NOT COM, J8 12V CIG. SOCKET, J9 5V LED STRIP, M1 ORIGINAL PSU FAN, SW1 MAINTAINED PS_ON, U1 ZK-4KX MODULE

Commit message: Update circuit
Parts:
- removed D1: GREEN / SB, symbol Project:LED
- removed D2: RED / PWR_OK, symbol Project:LED
- removed F1, F2, F3, F4: Fuse, symbol Project:Fuse
- removed J1: ATX SIGNAL MAP ONLY, symbol Project:ATX24_LOGICAL
- removed J8: 12V CIG. SOCKET, symbol Project:Load2
- removed J9: 5V LED STRIP, symbol Project:Load2
- removed M1: ORIGINAL PSU FAN, symbol Project:FanAssembly
- removed R1, R2: 1k, symbol Project:R
- removed SW1: MAINTAINED PS_ON, symbol Project:Switch
- added D1: GREEN / STANDBY, symbol Device:LED
- added D2: RED / POWER GOOD, symbol Device:LED
- added F1, F2, F3, F4: Fuse, symbol Device:Fuse
- added J1: PLENTY ATX500WS, symbol Project:ATX_PSU
- added J8: 12 V CIG. SOCKET, symbol Project:Socket
- added J9: 5 V LED STRIP, symbol Project:LED_Strip
- added M1: Internal PSU fan, symbol Project:InternalFan
- added R1, R2: 1k, symbol Device:R
- added SW1: MAIN ON/OFF, symbol Switch:SW_SPST
- J2: value RED +12V -> 12 V / RED
- J3: value YELLOW +5V -> 5 V / YELLOW
- J4: value GREEN +3.3V -> 3.3 V / GREEN
- J5: value BLACK COM -> GND / BLACK
- J6: value ADJ + -> ADJ + / RED
- J7: value ADJ - / NOT COM -> ADJ - / BLACK
- TP1: value PWR_OK TEST -> PWR_OK
- U1: value ZK-4KX MODULE -> ZK-4KX
Connections:
- net COM: now also D1.1 (K), D2.1 (K), J1.15 (COM), J1.17 (COM), J1.18 (COM), J1.19 (COM), J1.24 (COM), J1.3 (COM), J1.5 (COM), J1.7 (COM), J8.2 (-), J9.2 (-), SW1.2 (B)
- net PWR_OK: now also J1.8 (PWR_OK), R2.1
- net +12V_POST: no longer names the net of J2.1
- net +12V_POST: now also F1.2
- net +12V_RAW renamed +12V
- net +12V: now also F1.1, J1.10 (+12 V), J1.11 (+12 V), J8.1 (+)
- net +3V3_POST: no longer names the net of J4.1
- net +3V3_POST: now also F3.2
- net +5V_POST: no longer names the net of J3.1
- net +5V_POST: now also F2.2
- net ADJ_CONV_POS: no longer names the net of U1.3 (OUT+)
- net ADJ_CONV_POS: now also F4.1
- net ADJ_NEG: no longer names the net of J7.1, U1.4 (OUT-)
- net ADJ_POS: no longer names the net of J6.1
- net ADJ_POS: now also F4.2
- new net: D2.2 (A), R2.2
- new net: J1.16 (PS_ON#), SW1.1 (A)
- new net: D1.2 (A), R1.2
- new net +3V3: F3.1, J1.1 (+3.3 V), J1.12 (+3.3 V), J1.13 (+3.3 V), J1.2 (+3.3 V)
- new net +5V: F2.1, J1.21 (+5 V), J1.22 (+5 V), J1.23 (+5 V), J1.4 (+5 V), J1.6 (+5 V), J9.1 (+)
- new net +5VSB: J1.9 (+5VSB), R1.1
Other:
- note added: "ADJUSTABLE OUTPUT"
- note added: "ATX BENCH POWER SUPPLY"
- note added: "ATX supply"
- note added: "Centre + / outer contact COM"
- note added: "External DC wiring"
- note added: "F1-F3: fixed outputs. F4: adjustable output path shown in the project drawing."
- note added: "FIXED OUTPUTS"
- note added: "J1: grouped equivalent pins from the standard 24-pin ATX signal map."
- note added: "PSU and converter internals are not shown. See report for fuse selection and PWR_OK loading."
- note added: "Standard signal pins"
- note removed: "A. ATX SUPPLY SIGNALS"
- note removed: "B. FIXED OUTPUTS / SEPARATE FUSES"
- note removed: "C. SOCKET, STRIP AND FAN"
- note removed: "D. ADJUSTABLE OUTPUT / SEPARATE RETURN"
- note removed: "D1: green, purple +5VSB wire. D2: red, gray PWR_OK wire."
- note removed: "DIY ATX BENCH POWER SUPPLY | REV 1.5"
- note removed: "E. MAIN SWITCH"
- note removed: "F. STANDBY AND MAIN INDICATORS"
- note removed: "F1: 12 V output F2: 5 V output F3: 3.3 V output Fixed outputs share the COM terminal."
- note removed: "Green indicates standby power; red follows PWR_OK. Signal loading and fuse selection: see report calculations."
- note removed: "J8: 12 V panel-mount cigarette-lighter power socket. Centre contact: +12 V. Outer contact: COM. J9: 5 V LED strip, direct PSU output supply. M1: original fan circuit inside PSU1."
- note removed: "PSU1: PLENTY COMPUTER ATX500WS. Pin numbers: standard 24-pin ATX signal reference. COM is the common supply return."
- note removed: "Project 1 - Electronics Circuits Laboratory"
- note removed: "SW1 closed: main outputs ON. SW1 open: main outputs OFF. Standby supply remains active while AC is connected."
- note removed: "U1: ZK-4KX buck-boost module. Load return connects to OUT-. Separate return; non-isolated output."
- title: DIY ATX Bench Power Supply -> ATX Bench Power Supply

Commit message: Update schematic
Parts:
- removed F4: Fuse, symbol Device:Fuse
Connections:
- net at U1.3 (OUT+): now also J6.1
Other:
- note added: "F1-F3: three fixed-output fuses. Adjustable OUT+ connects directly to its terminal."
- note removed: "F1-F3: fixed outputs. F4: adjustable output path shown in the project drawing."

Commit message: Remove unused test point
Parts:
- removed TP1: PWR_OK, symbol Project:Post
